File: comixino/hw/comixino/comixino.kicad_pcb (KiCad board)
At the start: 2 copper layers, 99 x 68 mm, 33 parts, among them J1 Conn_01x02, J10 Conn_01x04, J11 Conn_02x03_Odd_Even, J12 Conn_02x03_Odd_Even, J2 Conn_01x02, J3 EXPANSION, J4 EXPANSION, J5 Conn_01x04, J6 Conn_01x06, J7 Conn_01x02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

Commit message: kicad
Parts:
- J1: footprint Connector_PinHeader_2.54mm:PinHeader_1x02_P2.54mm_Vertical -> Connector_PinHeader_2.54mm:PinHeader_1x02_P2.54mm_Horizontal
- J11, J12: footprint Connector_PinHeader_2.54mm:PinHeader_2x03_P2.54mm_Vertical -> Connector_PinHeader_2.54mm:PinHeader_2x03_P2.54mm_Horizontal
- J8: footprint Connector_PinHeader_2.54mm:PinHeader_1x03_P2.54mm_Vertical -> Connector_PinHeader_2.54mm:PinHeader_1x03_P2.54mm_Horizontal
Other:
- board text added: "100"
- board text added: "500"
- board text added: "GND VCC MISO MOSI SCK CS"
- board text added: "GND VCC SCL SDA"
